File: hardwire/two-phase/two-phase_GND_OLD.kicad_pcb (KiCad board)
At the start: 2 copper layers, 157.8 x 153.8 mm, 176 parts, among them J1 Conn_01x08_Female, J2 Conn_01x01_Female, J3 Conn_01x01_Female, J4 Conn_01x01_Female, J5 Conn_01x01_Female, J6 Conn_01x01_Female, J7 Conn_01x01_Female, Q1 BC849, Q10 BC849, Q11 IRF3205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

Commit message: update pcb, generate gerber
Routing:
- net GND: track 0.55 -> 1498.2 mm
- net +5V: track 600.2 -> 603.6 mm
- net /OUT_PH_2_A: track 116.2 -> 118.3 mm
- net +12V: track 544.5 -> 545.6 mm
